Commit message: algorithm for yaw angle and aruco material

File: model/aruco_robot.xacro (robot description, xacro)
@@ -50,5 +50,5 @@
   </link>
   <gazebo reference="base">
-    <material>Gazebo/Blue</material>
+    <material>aruco/material</material>
   </gazebo>
   <link name="tcp">

Commit message: dae model

File: model/aruco_robot.xacro (robot description, xacro)
@@ -1,6 +1,7 @@
 <?xml version="1.0"?>
 <robot xmlns:xacro="http://www.ros.org/wiki/xacro" name="aruco_robot">
-  <xacro:property name="base_x" value="1.0"/>
-  <xacro:property name="base_y" value="1.0"/>
+  <xacro:property name="M_PI" value="3.1415926"/>
+  <xacro:property name="base_x" value="0.5"/>
+  <xacro:property name="base_y" value="0.5"/>
   <xacro:property name="base_z" value="0.05"/>
   <xacro:property name="link_xy" value="0.05"/>
@@ -30,7 +31,13 @@
       </geometry>
     </collision>
+    <visual>
+      <origin xyz="0.0 0.0 ${base_z/2}" rpy="0.0 0.0 0.0"/>
+      <geometry>
+        <mesh filename="package://my_aruco/model/board_0.dae"/>
+      </geometry>
+    </visual>
     <inertial>
-      <mass value="5"/>
-      <inertia ixx="0.1" ixy="0.0" ixz="0.0" iyy="0.1" iyz="0.0" izz="0.1"/>
+      <mass value="100"/>
+      <inertia ixx="10" ixy="0.0" ixz="0.0" iyy="10" iyz="0.0" izz="10"/>
     </inertial>
     <!-- link -->
@@ -67,5 +74,5 @@
     </collision>
     <inertial>
-      <mass value="0.2"/>
+      <mass value="0.1"/>
       <inertia ixx="0.01" ixy="0.0" ixz="0.0" iyy="0.005" iyz="0.0" izz="0.005"/>
     </inertial>
@@ -80,3 +87,35 @@
     <origin xyz="0.0 0.0 ${link_z}" rpy="0 0 0"/>
   </joint>
+  <gazebo reference="tcp">
+    <sensor name="tcp_camera" type="camera" update_rate="30">
+      <origin xyz="0.0 0.0 0.0" rpy="0.0 0.0 {M_PI/2}"/>
+      <always_on>true</always_on>
+      <camera>
+        <horizental_fov>1.5707</horizental_fov>
+        <image>
+          <width>640</width>
+          <height>480</height>
+          <format>RGB8</format>
+        </image>
+        <clip>
+          <near>0.01</near>
+          <far>8.0</far>
+        </clip>
+      </camera>
+      <plugin name="camera_camera_controller" filename="libgazebo_ros_camera.so">
+        <alwaysOn>true</alwaysOn>
+        <updateRate>0.0</updateRate>
+        <cameraName>arm_sensor/camera</cameraName>
+        <imageTopicName>image_raw</imageTopicName>
+        <cameraInfoTopicName>camera_info</cameraInfoTopicName>
+        <frameName>camera_link</frameName>
+        <hackBaseline>0.07</hackBaseline>
+        <distortionK1>0.0</distortionK1>
+        <distortionK2>0.0</distortionK2>
+        <distortionK3>0.0</distortionK3>
+        <distortionT1>0.0</distortionT1>
+        <distortionT2>0.0</distortionT2>
+      </plugin>
+    </sensor>
+  </gazebo>
 </robot>

Commit message: evaluation

File: model/aruco_robot.xacro (robot description, xacro)
@@ -6,5 +6,5 @@
   <xacro:property name="base_z" value="0.05"/>
   <xacro:property name="link_xy" value="0.05"/>
-  <xacro:property name="link_z" value="1.5"/>
+  <xacro:property name="link_z" value="0.5"/>
   <xacro:property name="tcp_x" value="0.1"/>
   <xacro:property name="tcp_y" value="0.1"/>
@@ -31,10 +31,4 @@
       </geometry>
     </collision>
-    <visual>
-      <origin xyz="0.0 0.0 ${base_z/2}" rpy="0.0 0.0 0.0"/>
-      <geometry>
-        <mesh filename="package://my_aruco/model/board_0.dae"/>
-      </geometry>
-    </visual>
     <inertial>
       <mass value="100"/>
@@ -42,5 +36,5 @@
     </inertial>
     <!-- link -->
-    <visual>
+    <!-- <visual>
       <origin xyz="${base_x/2} 0.0 ${link_z/2}" rpy="0.0 0.0 0.0"/>
       <geometry>
@@ -48,5 +42,5 @@
       </geometry>
       <material name="blue"/>
-    </visual>
+    </visual> -->
     <collision>
       <origin xyz="${base_x/2} 0.0 ${link_z/2}" rpy="0.0 0.0 0.0"/>
@@ -56,10 +50,23 @@
     </collision>
   </link>
+  <link name="board">
+    <visual>
+      <origin xyz="0.0 0.0 ${base_z/2}" rpy="0.0 0.0 0.0"/>
+      <geometry>
+        <mesh filename="package://my_aruco/model/board_0.dae"/>
+      </geometry>
+    </visual>
+  </link>
+  <joint name="joint_base_board" type="fixed">
+    <parent link="base"/>
+    <child link="board"/>
+    <!-- <origin xyz="0.0 0.0 ${link_z}" rpy="0 0 0"/> -->
+  </joint>
   <gazebo reference="base">
-    <material>aruco/material</material>
+    <material>Gazebo/Gray</material>
   </gazebo>
   <link name="tcp">
     <visual>
-      <origin xyz="0.0 0.0 0.0" rpy="0.0 0.0 0.0"/>
+      <origin xyz="0.0 0.0 0.0" rpy="0.0 ${M_PI/2} 0.0"/>
       <geometry>
         <box size="${tcp_x} ${tcp_z} ${tcp_y}"/>
@@ -84,10 +91,9 @@
     <parent link="base"/>
     <child link="tcp"/>
-    <axis xyz="1 0 0"/>
-    <origin xyz="0.0 0.0 ${link_z}" rpy="0 0 0"/>
+    <axis xyz="0 0 1"/>
+    <origin xyz="0.0 0.0 ${link_z}" rpy="0 ${M_PI/2} 0"/>
   </joint>
   <gazebo reference="tcp">
     <sensor name="tcp_camera" type="camera" update_rate="30">
-      <origin xyz="0.0 0.0 0.0" rpy="0.0 0.0 {M_PI/2}"/>
       <always_on>true</always_on>
       <camera>
@@ -119,3 +125,18 @@
     </sensor>
   </gazebo>
+  <transmission name="tran1">
+    <type>transmission_interface/SimpleTransmission</type>
+    <joint name="joint_base_board">
+      <hardwareInterface>EffortJointInterface</hardwareInterface>
+    </joint>
+    <actuator name="motor1">
+      <hardwareInterface>EffortJointInterface</hardwareInterface>
+      <mechanicalReduction>1</mechanicalReduction>
+    </actuator>
+  </transmission>
+  <gazebo>
+    <plugin name="gazebo_ros_control" filename="libgazebo_ros_control.so">
+      <robotNamespace>/rrbot</robotNamespace>
+    </plugin>
+  </gazebo>
 </robot>

Commit message: gazebo

File: model/aruco_robot.xacro (robot description, xacro)
@@ -112,5 +112,5 @@
         <alwaysOn>true</alwaysOn>
         <updateRate>0.0</updateRate>
-        <cameraName>arm_sensor/camera</cameraName>
+        <cameraName>camera</cameraName>
         <imageTopicName>image_raw</imageTopicName>
         <cameraInfoTopicName>camera_info</cameraInfoTopicName>
@@ -125,11 +125,11 @@
     </sensor>
   </gazebo>
-  <transmission name="tran1">
+  <transmission name="tcp_joint_trans">
     <type>transmission_interface/SimpleTransmission</type>
-    <joint name="joint_base_board">
-      <hardwareInterface>EffortJointInterface</hardwareInterface>
+    <joint name="joint_base_tcp">
+      <hardwareInterface>hardware_interface/EffortJointInterface</hardwareInterface>
     </joint>
-    <actuator name="motor1">
-      <hardwareInterface>EffortJointInterface</hardwareInterface>
+    <actuator name="tcp_joint_motor">
+      <hardwareInterface>hardware_interface/EffortJointInterface</hardwareInterface>
       <mechanicalReduction>1</mechanicalReduction>
     </actuator>
@@ -137,5 +137,5 @@
   <gazebo>
     <plugin name="gazebo_ros_control" filename="libgazebo_ros_control.so">
-      <robotNamespace>/rrbot</robotNamespace>
+      <robotNamespace>/aruco_robot</robotNamespace>
     </plugin>
   </gazebo>
