Commit message: new model and gt of slamdog sim

File: urdf/slamdog/slamdog.xacro (robot description, xacro)
@@ -9,7 +9,8 @@
     <xacro:property name="wheel_length" value="0.1"/>
     <xacro:property name="wheel_radius" value="0.3"/>
-    <xacro:property name="distance" value="1.5"/>
+    <xacro:property name="distance" value="1.0"/>
     <xacro:property name="link_width" value="0.05"/>
-    <xacro:property name="move" value="0.3"/>
+    <xacro:property name="move_y" value="0.3"/>
+    <xacro:property name="move_z" value="0.1"/>
     <xacro:property name="installation_position" value="-${x_length/2 + 0.05}"/>
     <material name="blue">
@@ -189,4 +190,21 @@
         </visual>
     </link>
+    <!-- board -->
+    <link name="board_2">
+        <visual>
+            <origin xyz="0.0 0.0 0.0}" rpy="0.0 ${M_PI/2} 0.0"/>
+            <geometry>
+                <mesh filename="package://my_aruco/urdf/markers/board_2.dae"/>
+            </geometry>
+        </visual>
+    </link>
+    <link name="board_3">
+        <visual>
+            <origin xyz="0.0 0.0 0.0}" rpy="0.0 ${M_PI/2} 0.0"/>
+            <geometry>
+                <mesh filename="package://my_aruco/urdf/markers/board_3.dae"/>
+            </geometry>
+        </visual>
+    </link>
     <!-- camera -->
     <link name="link_camera">
@@ -231,5 +249,5 @@
     </joint>
     <joint name="fix_board_0" type="fixed">
-        <origin xyz="${-distance+x_length/2} ${move} 0.0" rpy="0.0 0.0 0.0"/>
+        <origin xyz="${-distance+x_length/2} ${move_y} -${z_length/2 - move_z}" rpy="0.0 0.0 0.0"/>
         <parent link="link_trailer"/>
         <child link="board_0"/>
@@ -237,7 +255,19 @@
     </joint>
     <joint name="fix_board_1" type="fixed">
-        <origin xyz="${-distance+x_length/2} ${-move} 0.0" rpy="0.0 0.0 0.0"/>
+        <origin xyz="${-distance+x_length/2} ${-move_y} -${z_length/2 - move_z}" rpy="0.0 0.0 0.0"/>
         <parent link="link_trailer"/>
         <child link="board_1"/>
+        <!-- <axis xyz="0.0 0.0 1.0"/> -->
+    </joint>
+    <joint name="fix_board_2" type="fixed">
+        <origin xyz="${-distance+x_length/2} ${move_y} ${z_length/2 - move_z}" rpy="0.0 0.0 0.0"/>
+        <parent link="link_trailer"/>
+        <child link="board_2"/>
+        <!-- <axis xyz="0.0 0.0 1.0"/> -->
+    </joint>
+    <joint name="fix_board_3" type="fixed">
+        <origin xyz="${-distance+x_length/2} ${-move_y} ${z_length/2 - move_z}" rpy="0.0 0.0 0.0"/>
+        <parent link="link_trailer"/>
+        <child link="board_3"/>
         <!-- <axis xyz="0.0 0.0 1.0"/> -->
     </joint>
@@ -287,4 +317,14 @@
         <actuator name="motor_right_wheel">
             <hardwareInterface>hardware_interface/VelocityJointInterface</hardwareInterface>
+            <mechanicalReduction>1</mechanicalReduction>
+        </actuator>
+    </transmission>
+    <transmission name="trans_trailer_joint">
+        <type>transmission_interface/SimpleTransmission</type>
+        <joint name="joint_trailer">
+            <hardwareInterface>hardware_interface/EffortJointInterface</hardwareInterface>
+        </joint>
+        <actuator name="motor_trailer">
+            <hardwareInterface>hardware_interface/EffortJointInterface</hardwareInterface>
             <mechanicalReduction>1</mechanicalReduction>
         </actuator>

Commit message: result eval

File: urdf/slamdog/slamdog.xacro (robot description, xacro)
@@ -9,9 +9,9 @@
     <xacro:property name="wheel_length" value="0.1"/>
     <xacro:property name="wheel_radius" value="0.3"/>
-    <xacro:property name="distance" value="1.0"/>
+    <xacro:property name="l1" value="0.4"/>
+    <xacro:property name="l2" value="1"/>
     <xacro:property name="link_width" value="0.05"/>
     <xacro:property name="move_y" value="0.3"/>
     <xacro:property name="move_z" value="0.1"/>
-    <xacro:property name="installation_position" value="-${x_length/2 + 0.05}"/>
     <material name="blue">
         <color rgba="0.0 0.5 1.0 1.0"/>
@@ -41,4 +41,38 @@
             </geometry>
         </collision>
+        <visual>
+            <origin xyz="-${l1/2} 0.0 -${z_length/2 - link_width/2}" rpy="0.0 0.0 0.0"/>
+            <geometry>
+                <box size="${l1} ${link_width}  ${link_width}"/>
+            </geometry>
+            <material name="blue"/>
+        </visual>
+        <!-- stable -->
+        <visual>
+            <origin xyz="${x_length/2 - link_width/2} 0.0 ${-z_length/4 - wheel_radius/2}" rpy="0.0 0.0 0.0"/>
+            <geometry>
+                <box size=" ${link_width}  ${link_width} ${wheel_radius - z_length/2}"/>
+            </geometry>
+            <material name="blue"/>
+        </visual>
+        <collision>
+            <origin xyz="${x_length/2 - link_width/2} 0.0 ${-z_length/4 - wheel_radius/2}" rpy="0.0 0.0 0.0"/>
+            <geometry>
+                <box size=" ${link_width}  ${link_width} ${wheel_radius - z_length/2}"/>
+            </geometry>
+        </collision>
+        <visual>
+            <origin xyz="-${x_length/2 - link_width/2} 0.0 ${-z_length/4 - wheel_radius/2}" rpy="0.0 0.0 0.0"/>
+            <geometry>
+                <box size=" ${link_width}  ${link_width} ${wheel_radius - z_length/2}"/>
+            </geometry>
+            <material name="blue"/>
+        </visual>
+        <collision>
+            <origin xyz="-${x_length/2 - link_width/2} 0.0 ${-z_length/4 - wheel_radius/2}" rpy="0.0 0.0 0.0"/>
+            <geometry>
+                <box size=" ${link_width}  ${link_width} ${wheel_radius - z_length/2}"/>
+            </geometry>
+        </collision>
         <inertial>
             <mass value="${mass}"/>
@@ -49,5 +83,5 @@
         <!-- body -->
         <visual>
-            <origin xyz="${-distance} 0.0 0.0" rpy="0.0 0.0 0.0"/>
+            <origin xyz="${-l2} 0.0 0.0" rpy="0.0 0.0 0.0"/>
             <geometry>
                 <box size="${x_length} ${y_length}  ${z_length}"/>
@@ -56,5 +90,5 @@
         </visual>
         <collision>
-            <origin xyz="${-distance} 0.0 0.0" rpy="0.0 0.0 0.0"/>
+            <origin xyz="${-l2} 0.0 0.0" rpy="0.0 0.0 0.0"/>
             <geometry>
                 <box size="${x_length} ${y_length}  ${z_length}"/>
@@ -63,21 +97,21 @@
         <!-- shaft -->
         <visual>
+            <origin xyz="-${link_width/2} 0.0 -${z_length/2 - link_width}" rpy="0.0 0.0 0.0"/>
+            <geometry>
+                <box size="${link_width} ${link_width}  ${link_width*2}"/>
+            </geometry>
+            <material name="orange"/>
+        </visual>
+        <!-- <collision>
             <origin xyz="0.0 0.0 -${z_length/2 - link_width}" rpy="0.0 0.0 0.0"/>
             <geometry>
                 <box size="${link_width} ${link_width}  ${link_width*2}"/>
             </geometry>
-            <material name="orange"/>
-        </visual>
-        <collision>
-            <origin xyz="0.0 0.0 -${z_length/2 - link_width}" rpy="0.0 0.0 0.0"/>
-            <geometry>
-                <box size="${link_width} ${link_width}  ${link_width*2}"/>
-            </geometry>
-        </collision>
+        </collision> -->
         <!-- link -->
         <visual>
-            <origin xyz="${-distance/2} 0.0 -${z_length/2 - link_width/2}" rpy="0.0 0.0 0.0"/>
-            <geometry>
-                <box size="${distance} ${link_width}  ${link_width}"/>
+            <origin xyz="${-l2/2} 0.0 -${z_length/2 - link_width/2}" rpy="0.0 0.0 0.0"/>
+            <geometry>
+                <box size="${l2} ${link_width}  ${link_width}"/>
             </geometry>
         </visual>
@@ -90,5 +124,5 @@
         <inertial>
             <mass value="${mass}"/>
-            <inertia ixx="1" ixy="0.0" ixz="0.0" iyy="1" iyz="0.0" izz="1"/>
+            <inertia ixx="1" ixy="0.0" ixz="0.0" iyy="1" iyz="0.0" izz="0.1"/>
         </inertial>
     </link>
@@ -231,5 +265,5 @@
     </joint>
     <joint name="joint_trailer_left_wheel" type="continuous">
-        <origin xyz="-${distance} ${y_length/2 + wheel_length/2} 0.0" rpy="0.0 0.0 0.0"/>
+        <origin xyz="-${l2} ${y_length/2 + wheel_length/2} 0.0" rpy="0.0 0.0 0.0"/>
         <parent link="link_trailer"/>
         <child link="link_trailer_left_wheel"/>
@@ -237,5 +271,5 @@
     </joint>
     <joint name="joint_trailer_right_wheel" type="continuous">
-        <origin xyz="-${distance} -${y_length/2 + wheel_length/2} 0.0" rpy="0.0 0.0 0.0"/>
+        <origin xyz="-${l2} -${y_length/2 + wheel_length/2} 0.0" rpy="0.0 0.0 0.0"/>
         <parent link="link_trailer"/>
         <child link="link_trailer_right_wheel"/>
@@ -243,5 +277,5 @@
     </joint>
     <joint name="joint_trailer" type="continuous">
-        <origin xyz="${installation_position} 0.0 0.0" rpy="0.0 0.0 0.0"/>
+        <origin xyz="-${l1} 0.0 0.0" rpy="0.0 0.0 0.0"/>
         <parent link="link_base"/>
         <child link="link_trailer"/>
@@ -249,5 +283,5 @@
     </joint>
     <joint name="fix_board_0" type="fixed">
-        <origin xyz="${-distance+x_length/2} ${move_y} -${z_length/2 - move_z}" rpy="0.0 0.0 0.0"/>
+        <origin xyz="${-l2+x_length/2} ${move_y} -${z_length/2 - move_z}" rpy="0.0 0.0 0.0"/>
         <parent link="link_trailer"/>
         <child link="board_0"/>
@@ -255,5 +289,5 @@
     </joint>
     <joint name="fix_board_1" type="fixed">
-        <origin xyz="${-distance+x_length/2} ${-move_y} -${z_length/2 - move_z}" rpy="0.0 0.0 0.0"/>
+        <origin xyz="${-l2+x_length/2} ${-move_y} -${z_length/2 - move_z}" rpy="0.0 0.0 0.0"/>
         <parent link="link_trailer"/>
         <child link="board_1"/>
@@ -261,5 +295,5 @@
     </joint>
     <joint name="fix_board_2" type="fixed">
-        <origin xyz="${-distance+x_length/2} ${move_y} ${z_length/2 - move_z}" rpy="0.0 0.0 0.0"/>
+        <origin xyz="${-l2+x_length/2} ${move_y} ${z_length/2 - move_z}" rpy="0.0 0.0 0.0"/>
         <parent link="link_trailer"/>
         <child link="board_2"/>
@@ -267,5 +301,5 @@
     </joint>
     <joint name="fix_board_3" type="fixed">
-        <origin xyz="${-distance+x_length/2} ${-move_y} ${z_length/2 - move_z}" rpy="0.0 0.0 0.0"/>
+        <origin xyz="${-l2+x_length/2} ${-move_y} ${z_length/2 - move_z}" rpy="0.0 0.0 0.0"/>
         <parent link="link_trailer"/>
         <child link="board_3"/>

Commit message: add docs and eval results

File: urdf/slamdog/slamdog.xacro (robot description, xacro)
@@ -14,4 +14,6 @@
     <xacro:property name="move_y" value="0.3"/>
     <xacro:property name="move_z" value="0.1"/>
+    <xacro:property name="friction" value="1.0"/>
+    <xacro:property name="wheel_mass" value="1.0"/>
     <material name="blue">
         <color rgba="0.0 0.5 1.0 1.0"/>
@@ -68,5 +70,5 @@
             </geometry>
             <material name="blue"/>
-        </visual>
+        </visual>K
         <collision>
             <origin xyz="-${x_length/2 - link_width/2} 0.0 ${-z_length/4 - wheel_radius/2}" rpy="0.0 0.0 0.0"/>
@@ -141,7 +143,15 @@
                 <cylinder radius="${wheel_radius}" length="${wheel_length}"/>
             </geometry>
-        </collision>
-        <inertial>
-            <mass value="0.5"/>
+            <surface>
+                <friction>
+                    <ode>
+                        <mu>${friction}</mu>
+                        <mu2>${friction}</mu2>
+                    </ode>
+                </friction>
+            </surface>
+        </collision>
+        <inertial>
+            <mass value="${wheel_mass}"/>
             <inertia ixx="0.01" ixy="0.0" ixz="0.0" iyy="0.005" iyz="0.0" izz="0.005"/>
         </inertial>
@@ -161,7 +171,15 @@
                 <cylinder radius="${wheel_radius}" length="${wheel_length}"/>
             </geometry>
-        </collision>
-        <inertial>
-            <mass value="0.5"/>
+            <surface>
+                <friction>
+                    <ode>
+                        <mu>${friction}</mu>
+                        <mu2>${friction}</mu2>
+                    </ode>
+                </friction>
+            </surface>
+        </collision>
+        <inertial>
+            <mass value="${wheel_mass}"/>
             <inertia ixx="0.01" ixy="0.0" ixz="0.0" iyy="0.005" iyz="0.0" izz="0.005"/>
         </inertial>

Commit message: remove useless files

File: urdf/slamdog/slamdog.xacro (robot description, xacro)
@@ -3,5 +3,4 @@
     xmlns:xacro="http://www.ros.org/wiki/xacro">
     <xacro:property name="M_PI" value="3.1415926"/>
-    <xacro:property name="mass" value="1"/>
     <xacro:property name="x_length" value="0.6"/>
     <xacro:property name="y_length" value="0.8"/>
@@ -9,11 +8,12 @@
     <xacro:property name="wheel_length" value="0.1"/>
     <xacro:property name="wheel_radius" value="0.3"/>
+    <xacro:property name="link_width" value="0.05"/>
     <xacro:property name="l1" value="0.4"/>
     <xacro:property name="l2" value="1"/>
-    <xacro:property name="link_width" value="0.05"/>
     <xacro:property name="move_y" value="0.3"/>
     <xacro:property name="move_z" value="0.1"/>
+    <xacro:property name="mass" value="1"/>
+    <xacro:property name="wheel_mass" value="1.0"/>
     <xacro:property name="friction" value="1.0"/>
-    <xacro:property name="wheel_mass" value="1.0"/>
     <material name="blue">
         <color rgba="0.0 0.5 1.0 1.0"/>
